File: protoflyer/electronics/plate-base/plate-base.kicad_sch (KiCad schematic)
At the start: 13 parts, among them J1 Conn_01x02_Socket, J10 Conn_01x02_Pin, J11 Conn_01x03_Pin, J2 Conn_01x02_Pin, J3 Conn_01x02_Pin, J4 Conn_01x02_Pin, J5 Conn_01x02_Pin, J6 Conn_01x03_Pin, J8 Conn_01x02_Pin, J9 Conn_01x02_Pin

Commit message: add explicit part number for AMASS connectors.
Parts:
- J1: Manufacturer No. (none) -> XT90PW-M
- J8, J9: Manufacturer No. (none) -> XT30UPB-F
Changed lines of the file:
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@@
 			)
 		)
-		(property "Manufacturer No." ""
+		(property "Manufacturer No." "XT30UPB-F"
 			(at 154.94 111.76 0)
 			(effects
@@
 			)
 		)
-		(property "Manufacturer No." ""
+		(property "Manufacturer No." "XT30UPB-F"
 			(at 154.94 93.98 0)
 			(effects
@@
 			)
 		)
-		(property "Manufacturer No." ""
+		(property "Manufacturer No." "XT90PW-M"
 			(at 115.57 97.79 0)
 			(effects
